File: LCD.kicad_sch (KiCad schematic)
At the start: 0 parts

Commit message: Everything is done except for the programming pins
Parts:
- added C15, C17: 100nF, symbol Device:C_Small_US
- added C16, C18: 1uF, symbol Device:C_Small_US
- added DS1: NHD-0216K1Z-NSW-BBW-L, NHD-0216K1Z-NSW-BBW-L:NHD_NHD-0216K1Z-NSW-BBW-L, symbol NHD-0216K1Z-NSW-BBW-L:NHD-0216K1Z-NSW-BBW-L
- added R11: 1.3kΩ, symbol Device:R_Small_US
- added R12, R13, R14, R8: 10kΩ, symbol Device:R_Small_US
- added R9: 3.7kΩ, symbol Device:R_Small_US
- added U6: SN74HCT245DWR, DW20, symbol SN4HCT245DR:SN74HCT245DWR
Connections:
- new net: R14.1, U6.11 (B8)
- new net: DS1.11_1 (DB4), U6.15 (B4)
- new net: DS1.12_1 (DB5), U6.14 (B5)
- new net: DS1.13_1 (DB6), U6.13 (B6)
- new net: DS1.14_1 (DB7), U6.12 (B7)
- new net: DS1.3_1 (V0), R11.1, R9.2
- new net: DS1.4_1 (RS), U6.16 (B3)
- new net: DS1.6_1 (E), U6.17 (B2)
- new net: R8.1, U6.18 (B1)
- new net: R13.1, U6.2 (A1)
- new net: R12.1, U6.9 (A8)
- new net +5V: C15.1, C16.1, C17.1, C18.1, DS1.15_1 (LED+), DS1.2_1 (VDD), R9.1, U6.1 (DIR), U6.20 (VCC)
- new net GND: C15.2, C16.2, C17.2, C18.2, DS1.16_1 (LED-), DS1.1_1 (VSS), DS1.S1 (SHIELD), DS1.S2 (SHIELD__1), DS1.S3 (SHIELD__2), DS1.S4 (SHIELD__3), R11.2, R12.2, R13.2, R14.2, R8.2, U6.10 (GND), U6.19 (*OE)
- new net LCD4: U6.5 (A4)
- new net LCD5: U6.6 (A5)
- new net LCD6: U6.7 (A6)
- new net LCD7: U6.8 (A7)
- new net LCD_E: U6.3 (A2)
- new net LCD_SR: U6.4 (A3)
- no-connect marks 0 -> 21

Commit message: Edits
Parts:
- C18: renamed from C17; footprint (none) -> Capacitor_SMD:C_01005_0402Metric
- C19: renamed from C18; footprint (none) -> Capacitor_SMD:C_01005_0402Metric
- C20: renamed from C15; footprint (none) -> Capacitor_SMD:C_01005_0402Metric
- C21: renamed from C16; footprint (none) -> Capacitor_SMD:C_01005_0402Metric
- R12: renamed from R13; footprint (none) -> Resistor_SMD:R_0402_1005Metric
- R13: renamed from R12; footprint (none) -> Resistor_SMD:R_0402_1005Metric
- R14: renamed from R8; footprint (none) -> Resistor_SMD:R_0402_1005Metric
- R15: renamed from R14; footprint (none) -> Resistor_SMD:R_0402_1005Metric
- R16: renamed from R9; footprint (none) -> Resistor_SMD:R_0402_1005Metric
- R17: renamed from R11; footprint (none) -> Resistor_SMD:R_0402_1005Metric
- renumbered DS1 to DS2, U6 to U7
